File: bycicle-speedometer-v2/bycicle-speedometer-v2.kicad_pcb (KiCad board)
At the start: 2 copper layers, 58 x 30 mm, 25 parts, among them J1 Conn_01x02_Pin, J2 Conn_01x02_Pin, J3 Conn_01x02_Pin, SW1 SW_Push_Dual, U1 ESP-12E, U2 AMS1117-3.3

Commit message: edited schematics
Parts:
- R5: value R -> 10k
- moved J2 3.73 mm to (199.2, 79.5), turned to -90 degrees
Connections:
- C1 pad 1: Net-(U1-VCC) -> 3V3
- U1 pad 8: Net-(U1-VCC) -> 3V3
Routing:
- net 3V3: track 0.00 -> 80.3 mm, vias 0 -> 2
- net Net-(D1-A): track 0.00 -> 60.5 mm
- net Net-(D1-K): track 0.00 -> 52.6 mm, vias 0 -> 1
- net Net-(D3-K): track 0.00 -> 50.4 mm, vias 0 -> 1
- net VCC: track 0.00 -> 13.3 mm
- net Net-(U1-REST): track 0.00 -> 13.2 mm
- net Sensor: track 0.00 -> 12.9 mm
- net Net-(J3-Pin_2): track 0.00 -> 10.1 mm
- net GND: track 0.00 -> 9.95 mm, vias 0 -> 4
- net Prog: track 0.00 -> 7.05 mm
- net led_c: track 0.00 -> 3.67 mm
- net led_a: track 0.00 -> 3.51 mm
- net led_b: track 0.00 -> 3.44 mm
- net Net-(U1-GPIO15): track 0.00 -> 1.88 mm
- net Net-(U1-CH_PD): track 0.00 -> 1.81 mm
- added copper zone on B.Cu, net GND
Other:
- outline, holes or cut-outs redrawn
- board text added: "+"
- board text added: "-"
- board text added: "Bicycle odometer"
- board text added: "FritzenLab.net FritzenLab.com.br"
- board text added: "Reed sensor"
