File: bycicle-speedometer-v2/bycicle-speedometer-v2.kicad_sch (KiCad schematic)
At the start: 23 parts, among them J1 Conn_01x02_Pin, J2 Conn_01x02_Pin, J3 Conn_01x02_Pin, J4 Conn_01x03_Pin, SW1 SW_Push_Dual, U1 ESP-12E

Commit message: added images and videos
Parts:
- C2: value 1u -> 100n
Changed lines of the file:
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@@
 			)
 		)
-		(property "Value" "1u"
+		(property "Value" "100n"
 			(at 96.52 107.9499 0)
 			(effects
